File: pcb/pcb.kicad_pcb (KiCad board)
At the start: 2 copper layers, 14 x 36 mm, 6 parts, among them J1 vik-module-connector, J2 Conn_01x05_Socket

Commit message: support VIK adapter
Connections:
- net BLUE renamed BLUE/SCK
- net GREEN renamed GREEN/CS
- net RED renamed RED/MOSI
- J1 pad 12: unconnected-(J1-3V3-Pad12) -> +3.3V
- J2 pad 3: unconnected-(J2-Pin_3-Pad3) -> +3.3V
Routing:
- net +3.3V: track 0.00 -> 30.0 mm, vias 0 -> 1
Other:
- board text added: "github.com/zzeneg led-view v0.2"
- board text removed: "github.com/zzeneg/led-view v0.2"
